File: kicad/modules/backplate/backplate.kicad_pcb (KiCad board)
At the start: 2 copper layers, 28 x 100 mm, 5 parts, among them J1 10018784-10210TLF

Commit message: backplate: update PCIe pins
Connections:
- J1 pad A1: unconnected-(J1-PadA1) -> CANP (x5)
- J1 pad A10: unconnected-(J1-PadA10) -> +3.3V (x5)
- J1 pad A11: unconnected-(J1-PadA11) -> +3.3V (x5)
- J1 pad A12: unconnected-(J1-PadA12) -> +5V (x5)
- J1 pad A13: unconnected-(J1-PadA13) -> +5V (x5)
- J1 pad A14: unconnected-(J1-PadA14) -> +5V (x5)
- J1 pad A16: unconnected-(J1-PadA16) -> +7.4V (x5)
- J1 pad A17: unconnected-(J1-PadA17) -> +7.4V (x5)
- J1 pad A18: unconnected-(J1-PadA18) -> +7.4V (x5)
- J1 pad A2: unconnected-(J1-PadA2) -> (no net) (x5)
- J1 pad A3: unconnected-(J1-PadA3) -> CANN (x5)
- J1 pad A4: unconnected-(J1-PadA4) -> GND (x5)
- J1 pad A5: unconnected-(J1-PadA5) -> GND (x5)
- J1 pad A6: unconnected-(J1-PadA6) -> GND (x5)
- J1 pad A7: unconnected-(J1-PadA7) -> GND (x5)
- J1 pad A9: unconnected-(J1-PadA9) -> +3.3V (x5)
- J1 pad B1: unconnected-(J1-PadB1) -> CANP (x5)
- J1 pad B10: unconnected-(J1-PadB10) -> +3.3V (x5)
- J1 pad B11: unconnected-(J1-PadB11) -> +3.3V (x5)
- J1 pad B12: unconnected-(J1-PadB12) -> +5V (x5)
- J1 pad B13: unconnected-(J1-PadB13) -> +5V (x5)
- J1 pad B14: unconnected-(J1-PadB14) -> +5V (x5)
- J1 pad B16: unconnected-(J1-PadB16) -> +7.4V (x5)
- J1 pad B17: unconnected-(J1-PadB17) -> +7.4V (x5)
- J1 pad B18: unconnected-(J1-PadB18) -> +7.4V (x5)
- J1 pad B2: unconnected-(J1-PadB2) -> (no net) (x5)
- J1 pad B3: unconnected-(J1-PadB3) -> CANN (x5)
- J1 pad B4: unconnected-(J1-PadB4) -> GND (x5)
- J1 pad B5: unconnected-(J1-PadB5) -> GND (x5)
- J1 pad B6: unconnected-(J1-PadB6) -> GND (x5)
- J1 pad B7: unconnected-(J1-PadB7) -> GND (x5)
- J1 pad B9: unconnected-(J1-PadB9) -> +3.3V (x5)

Commit message: backplate: finish initial revision
Parts:
- added R1: 120, Resistor_SMD:R_0805_2012Metric, F.Cu at (127.3, 54.0)
- added R2: 120, Resistor_SMD:R_0805_2012Metric, F.Cu at (127.3, 147.0)
Routing:
- net CANP: track 0.00 -> 98.4 mm
- net CANN: track 0.00 -> 98.4 mm
- net GND: vias 0 -> 60
- net +7.4V: vias 0 -> 12
- net +5V: vias 0 -> 12
- net +3.3V: vias 0 -> 12
- added copper zone on B.Cu, net +3.3V
- added copper zone on F.Cu, net +3.3V
- added copper zone on B.Cu, net +5V
- added copper zone on F.Cu, net +5V
- added copper zone on B.Cu, net +7.4V
- added copper zone on F.Cu, net +7.4V
- added copper zone on B.Cu, net GND
- added copper zone on F.Cu, net GND
Other:
- board text added: "backplate 0.1.0"
