File: kicad/modules/powersim/powersim.kicad_sch (KiCad schematic)
At the start: 2 parts, among them J1 Bus_PCI_Express_x1, J6 USB_C_Receptacle_USB2.0_16P

Commit message: powersim: add all components to schematic
Parts:
- added C1: 10u, symbol Device:C
- added C2: 100n, symbol Device:C
- added C3, C4: 22u, symbol Device:C
- added L1: 6.8u, symbol Device:L
- added U1: AP63203WU, Package_TO_SOT_SMD:TSOT-23-6, symbol Regulator_Switching:AP63203WU
Connections:
- net +3.3V: now also C3.1, C4.1, L1.2, U1.1 (FB)
- net +5V: now also C1.1, U1.2 (EN), U1.3 (IN)
- net GND: now also C1.2, C3.2, C4.2, U1.4 (GND)
- removed net +7.4V: J1.A16 (PERp0), J1.A17 (PERn0), J1.A18 (GND), J1.B16 (GND), J1.B17 (~{PRSNT2}), J1.B18 (GND)
- new net: C2.2, L1.1, U1.5 (SW)
- new net: C2.1, U1.6 (BST)
- no-connect marks 13 -> 19
Other:
- note added: "Power sim module 0.1.0"
- note removed: "Sensor module 0.1.0"
